Commit message: FINISHED add camera and imu

File: ws/src/spider/urdf/Robot.urdf (robot description, URDF)
Before this commit: robot Robot, 34 links, 33 joints
Links:
- link l_Spider_base001: mass 0.04 -> None

File: ws/src/spider/urdf/Robot_sensors.urdf.xacro (robot description, xacro)
@@ -1,3 +1,79 @@
 <?xml version="1.0"?>
 <robot xmlns:xacro="http://www.ros.org/wiki/xacro">
+<!--IMU SENSOR-->
+<xacro:macro name="imu_sensor_structure" params="conex_link">
+    <link name="imu_link">
+    </link>
+    <joint name="imu_link_joint" type="fixed">
+        <parent link="${conex_link}"/>
+        <child link="imu_link"/>
+        <origin xyz="0 0 0" rpy="0 0 0"/>
+    </joint>
+  <gazebo reference="imu_link">
+    <sensor name="imu_sensor" type="imu">
+      <always_on>1</always_on>
+      <update_rate>30</update_rate>
+      <topic>/imu_sensor/data</topic>
+    </sensor>
+  </gazebo>
+</xacro:macro>
+<!--CAMERA SENSOR-->
+<xacro:macro name="camera_structure" params="conex1_link h_fov v_width v_height">
+    <link name="base_camera_front_link">
+        <visual>
+            <geometry>
+                <cylinder length="0.005" radius="0.001"/>
+            </geometry>
+        </visual>
+        <collision>
+            <geometry>
+                <cylinder length="0.005" radius="0.01"/>
+            </geometry>
+        </collision>
+    </link>
+    <joint name="base_camera_front_joint" type="fixed">
+        <origin rpy="0.00000 0.00000 0.00000" xyz="0.0065 0.0 0.005"/>
+        <parent link="${conex1_link}"/>
+        <child link="base_camera_front_link"/>
+    </joint>
+    <link name="camera_front_frame">
+    </link>
+    <joint name="camera_front_frame_joint" type="fixed">
+        <origin rpy="0.00000 0.00000 0.00000" xyz="0.00000 0.00000 0.00000"/>
+        <parent link="base_camera_front_link"/>
+        <child link="camera_front_frame"/>
+    </joint>
+    <link name="camera_optical_front">
+    </link>
+    <joint name="camera_front_link_joint" type="fixed">
+        <origin rpy="-1.57000 0.00000 -1.57000" xyz="0.00000 0.00000 0.00000"/>
+        <parent link="camera_front_frame"/>
+        <child link="camera_optical_front"/>
+    </joint>
+    <gazebo reference="camera_front_frame">
+        <sensor name="camera_front_sensor" type="camera">
+        <visualize>true</visualize>
+        <update_rate>30</update_rate>
+        <topic>/camera_front/image</topic>
+        <camera>
+            <horizontal_fov>${h_fov}</horizontal_fov>
+            <image>
+            <width>${v_width}</width>
+            <height>${v_height}</height>
+            <format>R8G8B8</format>
+            </image>
+            <clip>
+            <near>0.10</near>
+            <far>15.0</far>
+            </clip>
+            <noise>
+            <type>gaussian</type>
+            <mean>0.0</mean>
+            <stddev>0.007</stddev>
+            </noise>
+            <optical_frame_id>camera_front_frame</optical_frame_id>
+        </camera>
+        </sensor>
+    </gazebo>
+</xacro:macro>
 </robot>

File: ws/src/spider/urdf/Robot_wrapper.urdf.xacro (robot description, xacro)
@@ -4,3 +4,5 @@
     <xacro:include filename="Robot.urdf"/>
     <xacro:include filename="Robot_sensors.urdf.xacro"/>
+    <xacro:imu_sensor_structure conex_link="l_SG_base001"/>
+    <xacro:camera_structure conex1_link="l_Spider_camera_module004" h_fov="1.047" v_width="1080" v_height="720"/>
 </robot>

Commit message: Done REP urdf adapt

File: ws/src/spider/urdf/Robot.urdf (robot description, URDF)
Before this commit: robot Robot, 34 links, 33 joints
Links:
- removed link l_Spider_base001
- added link base_footprint
- added link base_link; collision box size=0.11317322158813477 0.11317322158813477 0.014693019866943359; visual mesh filename=package://spider/meshes/robotcad_simple_parts_spider_base_m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
Joints:
- removed joint l_Spider_base001__to__l_SG_base001
- removed joint l_Spider_base001__to__l_Spider_hip_backleft001
- removed joint l_Spider_base001__to__l_Spider_hip_backright001
- removed joint l_Spider_base001__to__l_Spider_hip_frontleft001
- removed joint l_Spider_base001__to__l_Spider_hip_frontright001
- removed joint l_Spider_base001__to__l_Spider_trail001
- added joint base_link__to__l_SG_base001: type fixed, parent base_link, child l_SG_base001, origin xyz=-0.016857 0.000684 0.0645 rpy=0 0 0
- added joint base_link__to__l_Spider_hip_backleft001: type fixed, parent base_link, child l_Spider_hip_backleft001, origin xyz=-0.02479 0.02499 0.05131 rpy=0 0 -2.356194490192345
- added joint base_link__to__l_Spider_hip_backright001: type fixed, parent base_link, child l_Spider_hip_backright001, origin xyz=-0.02479 -0.02357 0.05131 rpy=0 0 -0.7853981633974484
- added joint base_link__to__l_Spider_hip_frontleft001: type fixed, parent base_link, child l_Spider_hip_frontleft001, origin xyz=0.02381 0.02462 0.05131 rpy=0 0 2.356194490192345
- added joint base_link__to__l_Spider_hip_frontright001: type fixed, parent base_link, child l_Spider_hip_frontright001, origin xyz=0.02381 -0.02321 0.05131 rpy=0 0 0.7853981633974484
- added joint base_link__to__l_Spider_trail001: type fixed, parent base_link, child l_Spider_trail001, origin xyz=-0.016857 0.000684 0.0565 rpy=0 0 0
- added joint base_to_footprint: type fixed, parent base_footprint, child base_link, origin xyz=0 0 0.075  rpy=0 0 0

Commit message: Adding new world

File: ws/src/spider/urdf/Robot.urdf (robot description, URDF)
Before this commit: robot Robot, 35 links, 34 joints
Links:
- link l_Spider_trail001: mass 0.044 -> 0.294

File: ws/src/spider/urdf/Robot_sensors.urdf.xacro (robot description, xacro)
@@ -1,79 +1,3 @@
 <?xml version="1.0"?>
 <robot xmlns:xacro="http://www.ros.org/wiki/xacro">
-<!--IMU SENSOR-->
-<xacro:macro name="imu_sensor_structure" params="conex_link">
-    <link name="imu_link">
-    </link>
-    <joint name="imu_link_joint" type="fixed">
-        <parent link="${conex_link}"/>
-        <child link="imu_link"/>
-        <origin xyz="0 0 0" rpy="0 0 0"/>
-    </joint>
-  <gazebo reference="imu_link">
-    <sensor name="imu_sensor" type="imu">
-      <always_on>1</always_on>
-      <update_rate>30</update_rate>
-      <topic>/imu_sensor/data</topic>
-    </sensor>
-  </gazebo>
-</xacro:macro>
-<!--CAMERA SENSOR-->
-<xacro:macro name="camera_structure" params="conex1_link h_fov v_width v_height">
-    <link name="base_camera_front_link">
-        <visual>
-            <geometry>
-                <cylinder length="0.005" radius="0.001"/>
-            </geometry>
-        </visual>
-        <collision>
-            <geometry>
-                <cylinder length="0.005" radius="0.01"/>
-            </geometry>
-        </collision>
-    </link>
-    <joint name="base_camera_front_joint" type="fixed">
-        <origin rpy="0.00000 0.00000 0.00000" xyz="0.0065 0.0 0.005"/>
-        <parent link="${conex1_link}"/>
-        <child link="base_camera_front_link"/>
-    </joint>
-    <link name="camera_front_frame">
-    </link>
-    <joint name="camera_front_frame_joint" type="fixed">
-        <origin rpy="0.00000 0.00000 0.00000" xyz="0.00000 0.00000 0.00000"/>
-        <parent link="base_camera_front_link"/>
-        <child link="camera_front_frame"/>
-    </joint>
-    <link name="camera_optical_front">
-    </link>
-    <joint name="camera_front_link_joint" type="fixed">
-        <origin rpy="-1.57000 0.00000 -1.57000" xyz="0.00000 0.00000 0.00000"/>
-        <parent link="camera_front_frame"/>
-        <child link="camera_optical_front"/>
-    </joint>
-    <gazebo reference="camera_front_frame">
-        <sensor name="camera_front_sensor" type="camera">
-        <visualize>true</visualize>
-        <update_rate>30</update_rate>
-        <topic>/camera_front/image</topic>
-        <camera>
-            <horizontal_fov>${h_fov}</horizontal_fov>
-            <image>
-            <width>${v_width}</width>
-            <height>${v_height}</height>
-            <format>R8G8B8</format>
-            </image>
-            <clip>
-            <near>0.10</near>
-            <far>15.0</far>
-            </clip>
-            <noise>
-            <type>gaussian</type>
-            <mean>0.0</mean>
-            <stddev>0.007</stddev>
-            </noise>
-            <optical_frame_id>camera_front_frame</optical_frame_id>
-        </camera>
-        </sensor>
-    </gazebo>
-</xacro:macro>
 </robot>

File: ws/src/spider/urdf/Robot_wrapper.urdf.xacro (robot description, xacro)
@@ -2,7 +2,5 @@
 <robot xmlns:xacro="http://www.ros.org/wiki/xacro" name="Robot">
     <xacro:arg name="config_controllers" default="$(find spider)/config/spider_controllers.yaml"/>
-    <xacro:include filename="Load_Robot.urdf"/>
+    <xacro:include filename="Robot.urdf"/>
     <xacro:include filename="Robot_sensors.urdf.xacro"/>
-    <xacro:imu_sensor_structure conex_link="l_SG_base001"/>
-    <xacro:camera_structure conex1_link="l_Spider_camera_module004" h_fov="1.047" v_width="1080" v_height="720"/>
 </robot>
