Commit message: Adding sensors

File: ws/src/spider/urdf/Robot_sensors.urdf.xacro (robot description, xacro)
@@ -1,3 +1,84 @@
 <?xml version="1.0"?>
 <robot xmlns:xacro="http://www.ros.org/wiki/xacro">
+    <!-- LIDAR -->
+    <link name="laser_link"/>
+    <joint name="base_link_to_laser" type="fixed">
+        <parent link="base_link"/>
+        <child link="laser_link"/>
+        <origin xyz="0 0 0.15" rpy="0 0 0"/>
+    </joint>
+    <gazebo reference="laser_link">
+        <sensor name="lidar_180" type="gpu_lidar">
+            <pose>0 0 0 0 0 0</pose>
+            <topic>/lidar_180/scan</topic>
+            <update_rate>20</update_rate>
+            <lidar>
+                <scan>
+                <horizontal>
+                    <samples>360</samples>
+                    <min_angle>-1.570796</min_angle>
+                    <max_angle>1.570796</max_angle>
+                </horizontal>
+                </scan>
+                <range>
+                <min>0.05</min>
+                <max>10.0</max>
+                <resolution>0.01</resolution>
+                </range>
+            </lidar>
+            <visualize>true</visualize>
+            <always_on>1</always_on>
+        </sensor>
+    </gazebo>
+    <!-- IMU -->
+    <link name="imu_link"/>
+    <joint name="base_link_to_imu" type="fixed">
+        <parent link="base_link"/>
+        <child link="imu_link"/>
+        <origin xyz="0 0 0.1" rpy="0 0 0"/>
+    </joint>
+    <gazebo reference="imu_link">
+        <sensor name="imu_sensor" type="imu">
+        <pose>0 0 0 0 0 0</pose>
+        <always_on>1</always_on>
+        <update_rate>50</update_rate>
+        <topic>/imu_sensor/data</topic>
+            <imu>
+                <angular_velocity>
+                <x>true</x><y>true</y><z>true</z>
+                </angular_velocity>
+                <linear_acceleration>
+                <x>true</x><y>true</y><z>true</z>
+                </linear_acceleration>
+            </imu>
+        </sensor>
+    </gazebo>
+    <!-- Camera -->
+    <link name="camera_link"/>
+    <joint name="base_link_to_camera" type="fixed">
+        <parent link="l_Spider_camera_module004"/>
+        <child link="camera_link"/>
+        <origin xyz="0.0 0 0.0" rpy="0 0 0"/>
+    </joint>
+    <gazebo reference="camera_link">
+        <sensor name="camera_front" type="camera">
+            <pose>0 0 0 0 0 0</pose>
+            <always_on>1</always_on>
+            <update_rate>30</update_rate>
+            <camera>
+                <horizontal_fov>1.047</horizontal_fov>
+                <image>
+                    <width>640</width>
+                    <height>480</height>
+                    <format>R8G8B8</format>
+                </image>
+                <clip>
+                    <near>0.1</near>
+                    <far>100</far>
+                </clip>
+            </camera>
+            <topic>/camera_front/image</topic>
+            <visualize>true</visualize>
+        </sensor>
+    </gazebo>
 </robot>

File: ws/src/spider/urdf/Robot_wrapper.urdf.xacro (robot description, xacro)
@@ -2,5 +2,5 @@
 <robot xmlns:xacro="http://www.ros.org/wiki/xacro" name="Robot">
     <xacro:arg name="config_controllers" default="$(find spider)/config/spider_controllers.yaml"/>
-    <xacro:include filename="Robot.urdf"/>
-    <xacro:include filename="Robot_sensors.urdf.xacro"/>
+    <xacro:include filename="$(find spider)/urdf/Robot.urdf"/>
+    <xacro:include filename="$(find spider)/urdf/Robot_sensors.urdf.xacro"/>
 </robot>
